Commit message: Update firmware v6.1.0

File: alicia_d_descriptions/urdf/Alicia_D_v5_6/Alicia_D_v5_6_gripper_100mm.urdf (robot description, URDF)
Before this commit: robot Alicia_D_v5_6_gripper_100mm, 10 links, 9 joints
Links:
- removed link gripper_center
- added link tool0; visual sphere radius=0.005
Joints:
- joint finger: child gripper_center -> tool0

File: alicia_d_descriptions/urdf/Alicia_D_v5_6/Alicia_D_v5_6_gripper_50mm.urdf (robot description, URDF)
Before this commit: robot Alicia_D_v5_6_gripper_50mm, 10 links, 9 joints
Links:
- removed link gripper_center
- added link tool0; visual sphere radius=0.005
Joints:
- joint finger: child gripper_center -> tool0

Commit message: Update the urdf direction

File: alicia_d_descriptions/urdf/Alicia_D_v5_6/Alicia_D_v5_6_gripper_100mm.urdf (robot description, URDF)
Before this commit: robot Alicia_D_v5_6_gripper_100mm, 10 links, 9 joints
Links:
- link Link1: mass 0.195233452997321 -> 0.195233495556057
- link Link2: mass 0.20703368934203 -> 0.207033693066089
- link Link3: mass 0.0845575626224312 -> 0.0845575651613574
- link Link4: mass 0.0653695946193964 -> 0.0653695951425785
- link Link5: mass 0.0507639007674356 -> 0.050763902309721
- link Link6: mass 0.123436287808883 -> 0.119820573151617
- link base_link: mass 0.733961424639881 -> 0.733961424954529
- link left_gripper: mass 0.025646111367227 -> 0.0256461121677845
- link right_gripper: mass 0.0256461131643355 -> 0.0256461121677874
Joints:
- joint Gripper: axis 0 0 -1 -> 0 0 1; origin xyz=-0.000200000000001033 -0.050497849845622 0.130979659620446 rpy=1.5707963267949 0 0 -> xyz=-0.000200000000001088 -0.050497849845622 0.130979659620446 rpy=1.5707963267949 0 3.14159265358979
- joint Joint1: axis -0.0397713509246861 0 0.999208806829496 -> 0 0 1; origin xyz=0 0 0.1295 rpy=0 -0.0397818431857344 0 -> xyz=0 0 0.1295 rpy=0 0 0
- joint Joint2: axis 0 0 -1 -> 0 0 1; limit lower=-1.57 upper=1.57 effort=5 velocity=12 -> lower=-2 upper=2 effort=5 velocity=12; origin xyz=0.00170499781414124 0 0.0428360815487805 rpy=1.5707963267949 -1.5707963267949 0 -> xyz=0 0 0.04287 rpy=1.5708 1.5708 0
- joint Joint3: axis 0 0 -1 -> 0 0 1; limit lower=-0.78 upper=3.14159 effort=5 velocity=12 -> lower=-0.5 upper=3.14159 effort=5 velocity=12; origin xyz=0.223671302741224 0.0226916129580064 -4.99999999962493E-05 rpy=0 0 -2.35619449019234 -> xyz=-0.22367 0.022492 -5E-05 rpy=0 0 2.3562
- joint Joint4: axis 0 0 -1 -> 0 0 1; limit lower=-2.7925 upper=2.7925 effort=5 velocity=12 -> lower=-2.79 upper=2.79 effort=5 velocity=12; origin xyz=0.00211000000000178 -0.0990000000000033 -0.0002000000000025 rpy=1.5707963267949 0 0 -> xyz=-0.00211 -0.099 0.0002 rpy=-1.5708 0 0
- joint Joint5: axis 0 0 1 -> 0 0 -1; origin xyz=0 -0.000500000000001193 0.12235 rpy=1.5707963267949 0 0 -> xyz=0 -0.0005 -0.12235 rpy=1.5708 0 -3.1416
- joint Joint6: limit lower=-3.14 upper=3.14 effort=5 velocity=12 -> lower=-3.14159 upper=3.14159 effort=5 velocity=12; origin xyz=-0.00384999999999935 0.0574999999999998 -0.00100000000000219 rpy=-1.5707963267949 0 0 -> xyz=-0.00385 -0.0575 0.001 rpy=1.5708 0 0
- joint finger: origin xyz=-0.0002 0 0.13048 rpy=0 0 0 -> xyz=-0.0002 0 0.13098 rpy=0 0 0
- joint right_finger: axis 0 0 1 -> 0 0 -1; origin xyz=-0.0002 0.050502 0.13098 rpy=-1.5708 0 0 -> xyz=-0.000199999999998035 0.050502150154378 0.130979659620446 rpy=-1.5707963267949 0 3.14159265358978

File: alicia_d_descriptions/urdf/Alicia_D_v5_6/Alicia_D_v5_6_gripper_50mm.urdf (robot description, URDF)
Before this commit: robot Alicia_D_v5_6_gripper_50mm, 10 links, 9 joints
Links:
- link Link1: mass 0.195233452997321 -> 0.195233453613076
- link Link2: mass 0.207033689183231 -> 0.207033693061784
- link Link3: mass 0.084557560592733 -> 0.0845575681430809
- link Link4: mass 0.0653695946194211 -> 0.0653695951968861
- link Link5: mass 0.0507639007674435 -> 0.0507639016868948
- link Link6: mass 0.130364885866405 -> 0.130364883211194
- link base_link: mass 0.733961424639881 -> 0.733961424024115
- link left_gripper: mass 0.0256461113672271 -> 0.025646112167786
- link right_gripper: mass 0.0256461131643356 -> 0.025646112167786
Joints:
- joint Gripper: axis 0 0 -1 -> 0 0 1; origin xyz=0.0002 -0.0255 0.13098 rpy=1.5708 0 0 -> xyz=0.000199999999998979 0.0254999999999971 -0.130979659620445 rpy=-1.5707963267949 0 -3.14159265358979
- joint Joint1: axis -0.0397713509246861 0 0.999208806829496 -> 0 0 1; origin xyz=0 0 0.1295 rpy=0 -0.0397818431857344 0 -> xyz=0 0 0.1295 rpy=0 0 0
- joint Joint2: axis 0 0 -1 -> 0 0 1; limit lower=-1.57 upper=1.57 effort=5 velocity=12 -> lower=-1.5708 upper=1.5708 effort=5 velocity=12; origin xyz=0.00170499781414124 0 0.0428360815487805 rpy=1.5707963267949 -1.5707963267949 0 -> xyz=0 0 0.04287 rpy=1.5708 1.5708 0
- joint Joint3: axis 0 0 -1 -> 0 0 1; limit lower=-0.78 upper=3.14159 effort=5 velocity=12 -> lower=-0.78 upper=3.14 effort=5 velocity=12; origin xyz=0.223671302741224 0.0226916129580064 -4.99999999962493E-05 rpy=0 0 -2.35619449019234 -> xyz=-0.22367 0.022492 -5E-05 rpy=0 0 2.3562
- joint Joint4: limit lower=-2.7925 upper=2.7925 effort=5 velocity=12 -> lower=-2.79 upper=2.79 effort=5 velocity=12; origin xyz=0.00211000000000178 -0.0990000000000033 -0.0002000000000025 rpy=1.5707963267949 0 0 -> xyz=-0.00211 -0.099 0.0002 rpy=-1.5708 0 -3.1416
- joint Joint5: axis 0 0 1 -> 0 0 -1; origin xyz=0 -0.000500000000001193 0.12235 rpy=1.5707963267949 0 0 -> xyz=0 -0.0005 0.12235 rpy=-1.5708 0 0
- joint Joint6: axis 0 0 -1 -> 0 0 1; origin xyz=-0.00384999999999935 0.0574999999999998 -0.00100000000000219 rpy=-1.5707963267949 0 0 -> xyz=-0.00385 -0.0575 0.001 rpy=-1.5708 0 0
- joint finger: origin xyz=0.0002 0 0.13098 rpy=0 0 0 -> xyz=0.0002 0 -0.13098 rpy=0 0 0
- joint right_finger: origin xyz=0.0002 0.0255 0.13098 rpy=-1.5708 0 0 -> xyz=0.0002 -0.0255 -0.13098 rpy=1.5708 0 0
